Commit message: Revise parameter organization
-Rename parameter files and namespaces
-Get camera position and orientation from tf data instead of parameters
-Remove the ALL attribute from the rosserial_add_client_target, so that the arduino code is not automatically build
-Update URDF to include the appropriate frames and positions

File: urdf/ghost_car.urdf.xacro (robot description, xacro)
@@ -1,11 +1,12 @@
 <?xml version="1.0"?>
 <robot name="ghost_car" xmlns:xacro="http://ros.org/wiki/xacro">
+<xacro:property name="pi" value="3.1415926536" />
 <!-- Car Dimensions -->
-<xacro:property name="length" value=".3" />
-<xacro:property name="width" value=".2" />
-<xacro:property name="height" value=".05" />
+<xacro:property name="wheelbase" value="0.260" />
+<xacro:property name="track_width" value="0.162" />
+<xacro:property name="car_height" value="0.08" />
 <!-- Colours -->
 <material name="blue">
-    <color rgba="0 0 .8 1"/>
+    <color rgba="0 0 0.8 1"/>
 </material>
 <material name="black">
@@ -16,20 +17,34 @@
 </material>
 <!-- Main body -->
+<link name="base_footprint"/>
 <link name="base_link">
     <visual>
       <geometry>
-        <box size="${length} ${width} ${height}"/>
+        <box size="${wheelbase} ${track_width} ${car_height}"/>
       </geometry>
-      <origin rpy="0 0 0" xyz="0 0 ${.5*height}"/>
+      <origin rpy="0 0 0" xyz="${0.5*wheelbase} 0 ${0.5*car_height}"/>
       <material name="blue"/>
     </visual>
 </link>
+<joint name="base_joint" type="fixed">
+  <origin xyz="0 0 0" rpy="0 0 0" />
+  <parent link="base_footprint"/>
+  <child link="base_link" />
+</joint>
 <!-- IMU -->
+<!-- Origin is at the corner with the labeled axis, on the lower surface-->
+<xacro:property name="imu_length" value="0.02" />
+<xacro:property name="imu_width" value="0.03" />
+<xacro:property name="imu_height" value="0.004" />
+<xacro:property name="imu_x" value="0.025" />
+<xacro:property name="imu_y" value="-0.032" />
+<xacro:property name="imu_z" value="0.079" />
+<xacro:property name="imu_yaw" value="0.0" />
 <link name="imu">
   <visual>
     <geometry>
-      <box size=".03 .03 .004"/>
+      <box size="${imu_length} ${imu_width} ${imu_height}"/>
     </geometry>
-    <origin rpy="0 0 0" xyz="0 0 0.002"/>
+    <origin rpy="0 0 0" xyz="${0.5*imu_length} ${-0.5*imu_width} ${0.5*imu_height}"/>
     <material name="black"/>
   </visual>
@@ -38,11 +53,18 @@
   <parent link="base_link"/>
   <child link="imu"/>
-  <origin xyz="0 0 ${height}"/>
+  <origin rpy="0 0 ${imu_yaw}" xyz="${imu_x} ${imu_y} ${imu_z}"/>
 </joint>
 <!-- Camera -->
+<xacro:property name="camera_length" value="0.030" />
+<xacro:property name="camera_width" value="0.029" />
+<xacro:property name="camera_height" value="0.029" />
+<xacro:property name="camera_x" value="0.15" />
+<xacro:property name="camera_y" value="0" />
+<xacro:property name="camera_z" value="0.165" />
+<xacro:property name="camera_pitch" value="0.02" />
 <link name="camera">
   <visual>
     <geometry>
-      <box size=".04 .04 .04"/>
+      <box size="${camera_length} ${camera_width} ${camera_height}"/>
     </geometry>
     <origin rpy="0 0 0" xyz="0 0 0"/>
@@ -53,5 +75,5 @@
   <parent link="base_link"/>
   <child link="camera"/>
-  <origin xyz="${.5*length - 0.02} 0 ${height + 0.02}"/>
+  <origin rpy="0 ${camera_pitch} 0" xyz="${camera_x} ${camera_y} ${camera_z}"/>
 </joint>
 </robot>

Commit message: Change scan frame, and scan bug fix
-Scanner frame is created on groundplane below camera
-Scans are published in scanner frame
-Fix scanner range calculation error
-Add debug messages to lane_detector_nodelet

File: urdf/ghost_car.urdf.xacro (robot description, xacro)
@@ -77,3 +77,12 @@
   <origin rpy="0 ${camera_pitch} 0" xyz="${camera_x} ${camera_y} ${camera_z}"/>
 </joint>
+<!-- Scanner from camera -->
+<!-- Origin is on the ground plane directly below the camera -->
+<link name="scanner">
+</link>
+<joint name="scanner_origin" type="fixed">
+  <parent link="camera"/>
+  <child link="scanner"/>
+  <origin rpy="0 ${-camera_pitch} 0" xyz="0 0 ${-camera_z}"/>
+</joint>
 </robot>

Commit message: Add EKF to fuse odometry with IMU
-Use robot_localization package
-Add variance parameters to odometry_integration

File: urdf/ghost_car.urdf.xacro (robot description, xacro)
@@ -17,6 +17,5 @@
 </material>
 <!-- Main body -->
-<link name="base_footprint"/>
-<link name="base_link">
+<link name="base_footprint">
     <visual>
       <geometry>
@@ -27,17 +26,19 @@
     </visual>
 </link>
-<joint name="base_joint" type="fixed">
-  <origin xyz="0 0 0" rpy="0 0 0" />
+<!-- Centre of Gravity -->
+<link name="cog"/>
+<joint name="cog_joint" type="fixed">
+  <origin xyz="${0.5*wheelbase} 0 ${0.5*car_height}" rpy="0 0 0" />
   <parent link="base_footprint"/>
-  <child link="base_link" />
+  <child link="cog" />
 </joint>
 <!-- IMU -->
-<!-- Origin is at the corner with the labeled axis, on the lower surface-->
+<!-- Origin is at the centre of board -->
 <xacro:property name="imu_length" value="0.02" />
 <xacro:property name="imu_width" value="0.03" />
 <xacro:property name="imu_height" value="0.004" />
-<xacro:property name="imu_x" value="0.025" />
-<xacro:property name="imu_y" value="-0.032" />
-<xacro:property name="imu_z" value="0.079" />
+<xacro:property name="imu_x" value="${wheelbase + 0.032}" />
+<xacro:property name="imu_y" value="0.0" />
+<xacro:property name="imu_z" value="0.038" />
 <xacro:property name="imu_yaw" value="0.0" />
 <link name="imu">
@@ -46,10 +47,10 @@
       <box size="${imu_length} ${imu_width} ${imu_height}"/>
     </geometry>
-    <origin rpy="0 0 0" xyz="${0.5*imu_length} ${-0.5*imu_width} ${0.5*imu_height}"/>
+    <origin rpy="0 0 0" xyz="0 0 0"/>
     <material name="black"/>
   </visual>
 </link>
 <joint name="imu_mount" type="fixed">
-  <parent link="base_link"/>
+  <parent link="base_footprint"/>
   <child link="imu"/>
   <origin rpy="0 0 ${imu_yaw}" xyz="${imu_x} ${imu_y} ${imu_z}"/>
@@ -73,5 +74,5 @@
 </link>
 <joint name="camera_mount" type="fixed">
-  <parent link="base_link"/>
+  <parent link="base_footprint"/>
   <child link="camera"/>
   <origin rpy="0 ${camera_pitch} 0" xyz="${camera_x} ${camera_y} ${camera_z}"/>

Commit message: Lane detector upgrades
-Large overhaul to lane detector node, inclding projection methods, image processing, organization, etc.
-Make lane detector parameters reconfigurable
-Add script for measuring the pose of the camera with a checkerboard

File: urdf/ghost_car.urdf.xacro (robot description, xacro)
@@ -62,6 +62,6 @@
 <xacro:property name="camera_x" value="0.15" />
 <xacro:property name="camera_y" value="0" />
-<xacro:property name="camera_z" value="0.165" />
-<xacro:property name="camera_pitch" value="0.02" />
+<xacro:property name="camera_z" value="0.1452" />
+<xacro:property name="camera_pitch" value="${11.008*pi/180.0}" />
 <link name="camera">
   <visual>

Commit message: Revise lane detection strategy, and output data format
-Use IMU orientation to adjust camera transformations
-Scan image row-wise, instead of radiating out from centre
-Output lane points as laserscan or 2D/3D pointcloud

File: urdf/ghost_car.urdf.xacro (robot description, xacro)
@@ -63,5 +63,5 @@
 <xacro:property name="camera_y" value="0" />
 <xacro:property name="camera_z" value="0.1452" />
-<xacro:property name="camera_pitch" value="${11.008*pi/180.0}" />
+<xacro:property name="camera_pitch" value="${9.00*pi/180.0}" />
 <link name="camera">
   <visual>
@@ -80,9 +80,9 @@
 <!-- Scanner from camera -->
 <!-- Origin is on the ground plane directly below the camera -->
-<link name="scanner">
+<link name="camera_ground">
 </link>
-<joint name="scanner_origin" type="fixed">
+<joint name="camera_ground_origin" type="fixed">
   <parent link="camera"/>
-  <child link="scanner"/>
+  <child link="camera_ground"/>
   <origin rpy="0 ${-camera_pitch} 0" xyz="0 0 ${-camera_z}"/>
 </joint>
